Commit message: Added macro to read config from yaml file. * Common compute lenght macro

File: ur_description/urdf/ur.common.xacro (robot description, xacro)
@@ -14,3 +14,80 @@
     </inertial>
   </xacro:macro>
+  <xacro:macro name="read_file" params="yaml_file">
+    <xacro:property name="__limits" value="${yaml_file['limits']}"/>
+    <xacro:property name="__dh_parameters" value="${yaml_file['dh_parameters']}"/>
+    <xacro:property name="__offsets" value="${yaml_file['offsets']}"/>
+    <xacro:property name="__inertia_parameters" value="${yaml_file['inertia_parameters']}" />
+    <!-- JOINTS LIMIT PARAMETERS -->
+    <xacro:property name="shoulder_pan_lower_limit" value="${__limits['shoulder_pan']['lower']}" scope="parent"/>
+    <xacro:property name="shoulder_pan_upper_limit" value="${__limits['shoulder_pan']['upper']}" scope="parent"/>
+    <xacro:property name="shoulder_pan_velocity_limit" value="${__limits['shoulder_pan']['velocity']}" scope="parent"/>
+    <xacro:property name="shoulder_pan_effort_limit" value="${__limits['shoulder_pan']['effort']}" scope="parent"/>
+    <xacro:property name="shoulder_lift_lower_limit" value="${__limits['shoulder_lift']['lower']}" scope="parent"/>
+    <xacro:property name="shoulder_lift_upper_limit" value="${__limits['shoulder_lift']['upper']}" scope="parent"/>
+    <xacro:property name="shoulder_lift_velocity_limit" value="${__limits['shoulder_lift']['velocity']}" scope="parent"/>
+    <xacro:property name="shoulder_lift_effort_limit" value="${__limits['shoulder_lift']['effort']}" scope="parent"/>
+    <xacro:property name="elbow_joint_lower_limit" value="${__limits['elbow_joint']['lower']}" scope="parent"/>
+    <xacro:property name="elbow_joint_upper_limit" value="${__limits['elbow_joint']['upper']}" scope="parent"/>
+    <xacro:property name="elbow_joint_velocity_limit" value="${__limits['elbow_joint']['velocity']}" scope="parent"/>
+    <xacro:property name="elbow_joint_effort_limit" value="${__limits['elbow_joint']['effort']}" scope="parent"/>
+    <xacro:property name="wrist_1_lower_limit" value="${__limits['wrist_1']['lower']}" scope="parent"/>
+    <xacro:property name="wrist_1_upper_limit" value="${__limits['wrist_1']['upper']}" scope="parent"/>
+    <xacro:property name="wrist_1_velocity_limit" value="${__limits['wrist_1']['velocity']}" scope="parent"/>
+    <xacro:property name="wrist_1_effort_limit" value="${__limits['wrist_1']['effort']}" scope="parent"/>
+    <xacro:property name="wrist_2_lower_limit" value="${__limits['wrist_2']['lower']}" scope="parent"/>
+    <xacro:property name="wrist_2_upper_limit" value="${__limits['wrist_2']['upper']}" scope="parent"/>
+    <xacro:property name="wrist_2_velocity_limit" value="${__limits['wrist_2']['velocity']}" scope="parent"/>
+    <xacro:property name="wrist_2_effort_limit" value="${__limits['wrist_2']['effort']}" scope="parent"/>
+    <xacro:property name="wrist_3_lower_limit" value="${__limits['wrist_3']['lower']}" scope="parent"/>
+    <xacro:property name="wrist_3_upper_limit" value="${__limits['wrist_3']['upper']}" scope="parent"/>
+    <xacro:property name="wrist_3_velocity_limit" value="${__limits['wrist_3']['velocity']}" scope="parent"/>
+    <xacro:property name="wrist_3_effort_limit" value="${__limits['wrist_3']['effort']}" scope="parent"/>
+    <!-- DH PARAMETERS -->
+    <xacro:property name="d1" value="${__dh_parameters['d1']}" scope="parent"/>
+    <xacro:property name="a2" value="${__dh_parameters['a2']}" scope="parent"/>
+    <xacro:property name="a3" value="${__dh_parameters['a3']}" scope="parent"/>
+    <xacro:property name="d4" value="${__dh_parameters['d4']}" scope="parent"/>
+    <xacro:property name="d5" value="${__dh_parameters['d5']}" scope="parent"/>
+    <xacro:property name="d6" value="${__dh_parameters['d6']}" scope="parent"/>
+    <!-- OFFSETS -->
+    <xacro:property name="shoulder_offset" value="${__offsets['shoulder_offset']}" scope="parent"/>
+    <xacro:property name="elbow_offset" value="${__offsets['elbow_offset']}" scope="parent"/>
+    <!-- INERTIA PARAMETERS -->
+    <!-- mass -->
+    <xacro:property name="base_mass" value="${__inertia_parameters['base_mass']}" scope="parent"/>
+    <xacro:property name="shoulder_mass" value="${__inertia_parameters['shoulder_mass']}" scope="parent"/>
+    <xacro:property name="upper_arm_mass" value="${__inertia_parameters['upper_arm_mass']}" scope="parent"/>
+    <xacro:property name="forearm_mass" value="${__inertia_parameters['forearm_mass']}" scope="parent"/>
+    <xacro:property name="wrist_1_mass" value="${__inertia_parameters['wrist_1_mass']}" scope="parent"/>
+    <xacro:property name="wrist_2_mass" value="${__inertia_parameters['wrist_2_mass']}" scope="parent"/>
+    <xacro:property name="wrist_3_mass" value="${__inertia_parameters['wrist_3_mass']}" scope="parent"/>
+    <!-- center of mass -->
+    <xacro:property name="__shoulder_cog" value="${__inertia_parameters['center_of_mass']['shoulder_cog']}"/>
+    <xacro:property name="__upper_arm_cog" value="${__inertia_parameters['center_of_mass']['upper_arm_cog']}"/>
+    <xacro:property name="__forearm_cog" value="${__inertia_parameters['center_of_mass']['forearm_cog']}"/>
+    <xacro:property name="__wrist_1_cog" value="${__inertia_parameters['center_of_mass']['wrist_1_cog']}"/>
+    <xacro:property name="__wrist_2_cog" value="${__inertia_parameters['center_of_mass']['wrist_2_cog']}"/>
+    <xacro:property name="__wrist_3_cog" value="${__inertia_parameters['center_of_mass']['wrist_3_cog']}"/>
+    <xacro:property name="shoulder_cog" value="${__shoulder_cog['x']} ${__shoulder_cog['y']} ${__shoulder_cog['z']}" scope="parent"/>
+    <xacro:property name="upper_arm_cog" value="${__upper_arm_cog['x']} ${__upper_arm_cog['y']} ${__upper_arm_cog['z']}" scope="parent"/>
+    <xacro:property name="forearm_cog" value="${__forearm_cog['x']} ${__forearm_cog['y']} ${__forearm_cog['z']}" scope="parent"/>
+    <xacro:property name="wrist_1_cog" value="${__wrist_1_cog['x']} ${__wrist_1_cog['y']} ${__wrist_1_cog['z']}" scope="parent"/>
+    <xacro:property name="wrist_2_cog" value="${__wrist_2_cog['x']} ${__wrist_2_cog['y']} ${__wrist_2_cog['z']}" scope="parent"/>
+    <xacro:property name="wrist_3_cog" value="${__wrist_3_cog['x']} ${__wrist_3_cog['y']} ${__wrist_3_cog['z']}" scope="parent"/>
+    <!-- cylinder radius -->
+    <xacro:property name="shoulder_radius" value="${__inertia_parameters['shoulder_radius']}" scope="parent"/>
+    <xacro:property name="upper_arm_radius" value="${__inertia_parameters['upper_arm_radius']}" scope="parent"/>
+    <xacro:property name="elbow_radius" value="${__inertia_parameters['elbow_radius']}" scope="parent"/>
+    <xacro:property name="forearm_radius" value="${__inertia_parameters['forearm_radius']}" scope="parent"/>
+    <xacro:property name="wrist_radius" value="${__inertia_parameters['wrist_radius']}" scope="parent"/>
+  </xacro:macro>
+  <xacro:macro name="compute_lenght" params="d1 a2 a3 d4 d5 d6 shoulder_offset elbow_offset">
+    <xacro:property name="shoulder_height" value="${d1}" scope="parent"/>
+    <xacro:property name="upper_arm_length" value="${-a2}" scope="parent"/>
+    <xacro:property name="forearm_length" value="${-a3}" scope="parent"/>
+    <xacro:property name="wrist_1_length" value="${d4 - elbow_offset - shoulder_offset}" scope="parent"/>
+    <xacro:property name="wrist_2_length" value="${d5}" scope="parent"/>
+    <xacro:property name="wrist_3_length" value="${d6}" scope="parent"/>
+  </xacro:macro>
 </robot>

Commit message: added parent scope to the cog parameters

File: ur_description/urdf/ur.common.xacro (robot description, xacro)
@@ -64,10 +64,10 @@
     <xacro:property name="wrist_3_mass" value="${__inertia_parameters['wrist_3_mass']}" scope="parent"/>
     <!-- center of mass -->
-    <xacro:property name="__shoulder_cog" value="${__inertia_parameters['center_of_mass']['shoulder_cog']}"/>
-    <xacro:property name="__upper_arm_cog" value="${__inertia_parameters['center_of_mass']['upper_arm_cog']}"/>
-    <xacro:property name="__forearm_cog" value="${__inertia_parameters['center_of_mass']['forearm_cog']}"/>
-    <xacro:property name="__wrist_1_cog" value="${__inertia_parameters['center_of_mass']['wrist_1_cog']}"/>
-    <xacro:property name="__wrist_2_cog" value="${__inertia_parameters['center_of_mass']['wrist_2_cog']}"/>
-    <xacro:property name="__wrist_3_cog" value="${__inertia_parameters['center_of_mass']['wrist_3_cog']}"/>
+    <xacro:property name="__shoulder_cog" value="${__inertia_parameters['center_of_mass']['shoulder_cog']}" scope="parent"/>
+    <xacro:property name="__upper_arm_cog" value="${__inertia_parameters['center_of_mass']['upper_arm_cog']}" scope="parent"/>
+    <xacro:property name="__forearm_cog" value="${__inertia_parameters['center_of_mass']['forearm_cog']}" scope="parent"/>
+    <xacro:property name="__wrist_1_cog" value="${__inertia_parameters['center_of_mass']['wrist_1_cog']}" scope="parent"/>
+    <xacro:property name="__wrist_2_cog" value="${__inertia_parameters['center_of_mass']['wrist_2_cog']}" scope="parent"/>
+    <xacro:property name="__wrist_3_cog" value="${__inertia_parameters['center_of_mass']['wrist_3_cog']}" scope="parent"/>
     <xacro:property name="shoulder_cog" value="${__shoulder_cog['x']} ${__shoulder_cog['y']} ${__shoulder_cog['z']}" scope="parent"/>
     <xacro:property name="upper_arm_cog" value="${__upper_arm_cog['x']} ${__upper_arm_cog['y']} ${__upper_arm_cog['z']}" scope="parent"/>
