Commit message: Use full kinematics parameters in description
the kinematics parameters can be retrieved from a calibration mechanism
to precisely represent the robot's kinematics.

File: ur_description/urdf/ur5_robot.urdf.xacro (robot description, xacro)
@@ -3,4 +3,5 @@
        name="ur5" >
   <xacro:arg name="joints_limits_params" default="$(find ur_description)/config/ur5/joints_limits_parameters.yaml"/>
+  <xacro:arg name="kinematics_file" default="$(find ur_description)/config/ur5/default_kinematics.yaml"/>
   <xacro:arg name="physical_params" default="$(find ur_description)/config/ur5/physical_parameters.yaml"/>
   <xacro:arg name="visual_params" default="$(find ur_description)/config/ur5/visual_parameters.yaml"/>
@@ -11,4 +12,5 @@
    <!-- arm -->
    <xacro:ur_robot prefix="" joints_limits_parameters_file="${load_yaml('$(arg joints_limits_params)')}"
+                             kinematics_file="${load_yaml('$(arg kinematics_file)')}"
                              physical_parameters_file="${load_yaml('$(arg physical_params)')}"
                              visual_parameters_file="${load_yaml('$(arg visual_params)')}"
