Commit message: merge geometry into the same xacro macro

File: ur_description/urdf/ur.geometry.xacro (robot description, xacro)
@@ -2,14 +2,11 @@
 <robot xmlns:xacro="http://wiki.ros.org/xacro">
 <!--
-  Author: Kelsey Hawkins
-  Contributers: Jimmy Da Silva, Ajit Krisshna N L, Muhammad Asif Rana
+  Author: Ludovic Delval
+  Contributor: Felix Messmer, Kelsey Hawkins, Jimmy Da Silva, Ajit Krisshna N L, Muhammad Asif Rana
 -->
-  <xacro:include filename="$(find ur_description)/urdf/ur.transmission.xacro" />
-  <xacro:include filename="$(find ur_description)/urdf/ur.gazebo.xacro" />
-  <xacro:include filename="$(find ur_description)/urdf/ur.common.xacro" />
-  <xacro:macro name="ur10_robot" params="prefix joints_limits_parameters_file
-                                                physical_parameters_file
-                                                visual_parameters_file
-                                                transmission_hw_interface:=hardware_interface/PositionJointInterface">
+ <xacro:include filename="$(find ur_description)/urdf/ur.transmission.xacro" />
+ <xacro:include filename="$(find ur_description)/urdf/ur.gazebo.xacro" />
+ <xacro:include filename="$(find ur_description)/urdf/ur.common.xacro" />
+ <xacro:macro name="ur_robot" params="prefix joints_limits_parameters_file physical_parameters_file visual_parameters_file transmission_hw_interface:=hardware_interface/PositionJointInterface">
     <xacro:read_file joints_limits_parameters_file="${joints_limits_parameters_file}"
                     physical_parameters_file="${physical_parameters_file}"
@@ -42,5 +39,5 @@
       <axis xyz="0 0 1" />
       <limit lower="${shoulder_pan_lower_limit}" upper="${shoulder_pan_upper_limit}"
-             effort="${shoulder_pan_effort_limit}" velocity="${shoulder_pan_velocity_limit}"/>
+          effort="${shoulder_pan_effort_limit}" velocity="${shoulder_pan_velocity_limit}"/>
       <dynamics damping="0.0" friction="0.0"/>
     </joint>
@@ -69,5 +66,5 @@
       <axis xyz="0 1 0" />
       <limit lower="${shoulder_lift_lower_limit}" upper="${shoulder_lift_upper_limit}"
-             effort="${shoulder_lift_effort_limit}" velocity="${shoulder_lift_velocity_limit}"/>
+        effort="${shoulder_lift_effort_limit}" velocity="${shoulder_lift_velocity_limit}"/>
       <dynamics damping="0.0" friction="0.0"/>
     </joint>
@@ -96,5 +93,5 @@
       <axis xyz="0 1 0" />
       <limit lower="${elbow_joint_lower_limit}" upper="${elbow_joint_upper_limit}"
-        effort="${elbow_joint_effort_limit}" velocity="${elbow_joint_velocity_limit}"/>/>
+        effort="${elbow_joint_effort_limit}" velocity="${elbow_joint_velocity_limit}"/>
       <dynamics damping="0.0" friction="0.0"/>
     </joint>
@@ -123,5 +120,5 @@
       <axis xyz="0 1 0" />
       <limit lower="${wrist_1_lower_limit}" upper="${wrist_1_upper_limit}"
-             effort="${wrist_1_effort_limit}" velocity="${wrist_1_velocity_limit}"/>/>
+        effort="${wrist_1_effort_limit}" velocity="${wrist_1_velocity_limit}"/>
       <dynamics damping="0.0" friction="0.0"/>
     </joint>

Commit message: fixed length and collision typos

File: ur_description/urdf/ur.geometry.xacro (robot description, xacro)
@@ -12,5 +12,5 @@
                     physical_parameters_file="${physical_parameters_file}"
                     visual_parameters_file="${visual_parameters_file}"/>
-    <xacro:compute_lenght d1="${d1}" a2="${a2}" a3="${a3}"
+    <xacro:compute_length d1="${d1}" a2="${a2}" a3="${a3}"
                           d4="${d4}" d5="${d5}" d6="${d6}"
                           shoulder_offset="${shoulder_offset}" elbow_offset="${elbow_offset}"/>
@@ -26,5 +26,5 @@
       <collision>
         <geometry>
-          <mesh filename="${base_colision_mesh}"/>
+          <mesh filename="${base_collision_mesh}"/>
         </geometry>
       </collision>
@@ -53,5 +53,5 @@
       <collision>
         <geometry>
-          <mesh filename="${shoulder_colision_mesh}"/>
+          <mesh filename="${shoulder_collision_mesh}"/>
         </geometry>
       </collision>
@@ -80,5 +80,5 @@
       <collision>
         <geometry>
-          <mesh filename="${upper_arm_colision_mesh}"/>
+          <mesh filename="${upper_arm_collision_mesh}"/>
         </geometry>
       </collision>
@@ -107,5 +107,5 @@
       <collision>
         <geometry>
-          <mesh filename="${forearm_colision_mesh}"/>
+          <mesh filename="${forearm_collision_mesh}"/>
         </geometry>
       </collision>
@@ -134,5 +134,5 @@
       <collision>
         <geometry>
-          <mesh filename="${wrist_1_colision_mesh}"/>
+          <mesh filename="${wrist_1_collision_mesh}"/>
         </geometry>
       </collision>
@@ -161,5 +161,5 @@
       <collision>
         <geometry>
-          <mesh filename="${wrist_2_colision_mesh}"/>
+          <mesh filename="${wrist_2_collision_mesh}"/>
         </geometry>
       </collision>
@@ -188,5 +188,5 @@
       <collision>
         <geometry>
-          <mesh filename="${wrist_3_colision_mesh}"/>
+          <mesh filename="${wrist_3_collision_mesh}"/>
         </geometry>
       </collision>
