Commit message: made changes to ur3 to use yaml config

File: ur_description/urdf/ur3.urdf.xacro (robot description, xacro)
@@ -7,47 +7,9 @@
   <xacro:include filename="$(find ur_description)/urdf/ur.gazebo.xacro" />
   <xacro:include filename="$(find ur_description)/urdf/ur.common.xacro" />
-  <xacro:macro name="ur3_robot" params="prefix joint_limited
-     shoulder_pan_lower_limit:=${-pi}    shoulder_pan_upper_limit:=${pi}
-     shoulder_lift_lower_limit:=${-pi}    shoulder_lift_upper_limit:=${pi}
-     elbow_joint_lower_limit:=${-pi}    elbow_joint_upper_limit:=${pi}
-     wrist_1_lower_limit:=${-pi}    wrist_1_upper_limit:=${pi}
-     wrist_2_lower_limit:=${-pi}    wrist_2_upper_limit:=${pi}
-     wrist_3_lower_limit:=${-pi}    wrist_3_upper_limit:=${pi}">
-    <!-- Inertia parameters -->
-    <xacro:property name="base_mass" value="2.0" />  <!-- This mass might be incorrect -->
-    <xacro:property name="shoulder_mass" value="2.0" />
-    <xacro:property name="upper_arm_mass" value="3.42" />
-    <xacro:property name="forearm_mass" value="1.26" />
-    <xacro:property name="wrist_1_mass" value="0.8" />
-    <xacro:property name="wrist_2_mass" value="0.8" />
-    <xacro:property name="wrist_3_mass" value="0.35" />
-    <!-- These parameters are borrowed from the urcontrol.conf file
-        but are not verified for the correct permutation.
-        The permutation was guessed by looking at the UR5 parameters.
-        Serious use of these parameters needs further inspection. -->
-    <xacro:property name="shoulder_cog" value="0.0 -0.02 0.0" />
-    <xacro:property name="upper_arm_cog" value="0.13 0.0 0.1157" />
-    <xacro:property name="forearm_cog" value="0.05 0.0 0.0238" />
-    <xacro:property name="wrist_1_cog" value="0.0 0.0 0.01" />
-    <xacro:property name="wrist_2_cog" value="0.0 0.0 0.01" />
-    <xacro:property name="wrist_3_cog" value="0.0 0.0 -0.02" />
-    <!-- Kinematic model -->
-    <!-- Properties from urcontrol.conf -->
-    <xacro:property name="d1" value="0.1519" />
-    <xacro:property name="a2" value="-0.24365" />
-    <xacro:property name="a3" value="-0.21325" />
-    <xacro:property name="d4" value="0.11235" />
-    <xacro:property name="d5" value="0.08535" />
-    <xacro:property name="d6" value="0.0819" />
-    <!-- Arbitrary offsets for shoulder/elbow joints -->
-    <xacro:property name="shoulder_offset" value="0.1198" />  <!-- measured from model -->
-    <xacro:property name="elbow_offset" value="-0.0925" /> <!-- measured from model -->
-    <!-- link lengths used in model -->
-    <xacro:property name="shoulder_height" value="${d1}" />
-    <xacro:property name="upper_arm_length" value="${-a2}" />
-    <xacro:property name="forearm_length" value="${-a3}" />
-    <xacro:property name="wrist_1_length" value="${d4 - elbow_offset - shoulder_offset}" />
-    <xacro:property name="wrist_2_length" value="${d5}" />
-    <xacro:property name="wrist_3_length" value="${d6}" />
+  <xacro:macro name="ur3_robot" params="prefix yaml_file">
+    <xacro:read_file yaml_file="${yaml_file}"/>
+    <xacro:compute_lenght d1="${d1}" a2="${a2}" a3="${a3}"
+                          d4="${d4}" d5="${d5}" d6="${d6}"
+                          shoulder_offset="${shoulder_offset}" elbow_offset="${elbow_offset}"/>
     <link name="${prefix}base_link" >
       <visual>
@@ -73,10 +35,6 @@
       <origin xyz="0.0 0.0 ${shoulder_height}" rpy="0.0 0.0 0.0" />
       <axis xyz="0 0 1" />
-      <xacro:unless value="${joint_limited}">
-        <limit lower="${-2.0 * pi}" upper="${2.0 * pi}" effort="330.0" velocity="2.16"/>
-      </xacro:unless>
-      <xacro:if value="${joint_limited}">
-        <limit lower="${shoulder_pan_lower_limit}" upper="${shoulder_pan_upper_limit}" effort="330.0" velocity="2.16"/>
-      </xacro:if>
+      <limit lower="${shoulder_pan_lower_limit}" upper="${shoulder_pan_upper_limit}"
+          effort="${shoulder_pan_effort_limit}" velocity="${shoulder_pan_velocity_limit}"/>
       <dynamics damping="0.0" friction="0.0"/>
     </joint>
@@ -104,10 +62,6 @@
       <origin xyz="0.0 ${shoulder_offset} 0.0" rpy="0.0 ${pi / 2.0} 0.0" />
       <axis xyz="0 1 0" />
-      <xacro:unless value="${joint_limited}">
-        <limit lower="${-2.0 * pi}" upper="${2.0 * pi}" effort="330.0" velocity="2.16"/>
-      </xacro:unless>
-      <xacro:if value="${joint_limited}">
-        <limit lower="${shoulder_lift_lower_limit}" upper="${shoulder_lift_upper_limit}" effort="330.0" velocity="2.16"/>
-      </xacro:if>
+      <limit lower="${shoulder_lift_lower_limit}" upper="${shoulder_lift_upper_limit}"
+        effort="${shoulder_lift_effort_limit}" velocity="${shoulder_lift_velocity_limit}"/>
       <dynamics damping="0.0" friction="0.0"/>
     </joint>
@@ -135,10 +89,6 @@
       <origin xyz="0.0 ${elbow_offset} ${upper_arm_length}" rpy="0.0 0.0 0.0" />
       <axis xyz="0 1 0" />
-      <xacro:unless value="${joint_limited}">
-        <limit lower="${-pi}" upper="${pi}" effort="150.0" velocity="3.15"/>
-      </xacro:unless>
-      <xacro:if value="${joint_limited}">
-        <limit lower="${elbow_joint_lower_limit}" upper="${elbow_joint_upper_limit}" effort="150.0" velocity="3.15"/>
-      </xacro:if>
+      <limit lower="${elbow_joint_lower_limit}" upper="${elbow_joint_upper_limit}"
+        effort="${elbow_joint_effort_limit}" velocity="${elbow_joint_velocity_limit}"/>
       <dynamics damping="0.0" friction="0.0"/>
     </joint>
@@ -166,10 +116,6 @@
       <origin xyz="0.0 0.0 ${forearm_length}" rpy="0.0 ${pi / 2.0} 0.0" />
       <axis xyz="0 1 0" />
-      <xacro:unless value="${joint_limited}">
-        <limit lower="${-2.0 * pi}" upper="${2.0 * pi}" effort="54.0" velocity="3.2"/>
-      </xacro:unless>
-      <xacro:if value="${joint_limited}">
-        <limit lower="${wrist_1_lower_limit}" upper="${wrist_1_upper_limit}" effort="54.0" velocity="3.2"/>
-      </xacro:if>
+      <limit lower="${wrist_1_lower_limit}" upper="${wrist_1_upper_limit}"
+        effort="${wrist_1_effort_limit}" velocity="${wrist_1_velocity_limit}"/>
       <dynamics damping="0.0" friction="0.0"/>
     </joint>
@@ -197,10 +143,6 @@
       <origin xyz="0.0 ${wrist_1_length} 0.0" rpy="0.0 0.0 0.0" />
       <axis xyz="0 0 1" />
-      <xacro:unless value="${joint_limited}">
-        <limit lower="${-2.0 * pi}" upper="${2.0 * pi}" effort="54.0" velocity="3.2"/>
-      </xacro:unless>
-      <xacro:if value="${joint_limited}">
-        <limit lower="${wrist_2_lower_limit}" upper="${wrist_2_upper_limit}" effort="54.0" velocity="3.2"/>
-      </xacro:if>
+      <limit lower="${wrist_2_lower_limit}" upper="${wrist_2_upper_limit}"
+             effort="${wrist_2_effort_limit}" velocity="${wrist_2_velocity_limit}"/>
       <dynamics damping="0.0" friction="0.0"/>
     </joint>
@@ -228,10 +170,6 @@
       <origin xyz="0.0 0.0 ${wrist_2_length}" rpy="0.0 0.0 0.0" />
       <axis xyz="0 1 0" />
-      <xacro:unless value="${joint_limited}">
-        <limit lower="${-2.0 * pi}" upper="${2.0 * pi}" effort="54.0" velocity="3.2"/>
-      </xacro:unless>
-      <xacro:if value="${joint_limited}">
-        <limit lower="${wrist_3_lower_limit}" upper="${wrist_3_upper_limit}" effort="54.0" velocity="3.2"/>
-      </xacro:if>
+      <limit lower="${wrist_3_lower_limit}" upper="${wrist_3_upper_limit}"
+             effort="${wrist_3_effort_limit}" velocity="${wrist_3_velocity_limit}"/>
       <dynamics damping="0.0" friction="0.0"/>
     </joint>

File: ur_description/urdf/ur3_robot.urdf.xacro (robot description, xacro)
@@ -2,15 +2,11 @@
 <robot xmlns:xacro="http://ros.org/wiki/xacro"
        name="ur3" >
-  <!-- common stuff -->
-  <xacro:include filename="$(find ur_description)/urdf/common.gazebo.xacro" />
-  <!-- ur3 -->
-  <xacro:include filename="$(find ur_description)/urdf/ur3.urdf.xacro" />
-  <!-- arm -->
-  <xacro:ur3_robot prefix="" joint_limited="false"/>
-  <link name="world" />
-  <joint name="world_joint" type="fixed">
-    <parent link="world" />
-    <child link = "base_link" />
-    <origin xyz="0.0 0.0 0.0" rpy="0.0 0.0 0.0" />
-  </joint>
+   <!-- common stuff -->
+   <xacro:arg name="yaml_config" default="$(find ur_description)/config/ur3_default.yaml"/>
+   <!-- common stuff -->
+   <xacro:include filename="$(find ur_description)/urdf/common.gazebo.xacro" />
+   <!-- ur3 -->
+   <xacro:include filename="$(find ur_description)/urdf/ur3.urdf.xacro" />
+   <!-- arm -->
+   <xacro:ur3_robot prefix="" yaml_file="${load_yaml('$(arg yaml_config)')}"/>
 </robot>

Commit message: Improve inertia approximation for UR3

File: ur_description/urdf/ur3.urdf.xacro (robot description, xacro)
@@ -13,4 +13,13 @@
         iyy="${0.0833333 * mass * (3 * radius * radius + length * length)}" iyz="0.0"
         izz="${0.5 * mass * radius * radius}" />
+    </inertial>
+  </xacro:macro>
+  <xacro:macro name="box_inertial" params="x y z mass *origin">
+    <inertial>
+      <mass value="${mass}" />
+      <xacro:insert_block name="origin" />
+      <inertia ixx="${0.0833333 * mass * (y*y + z*z)}" ixy="0.0" ixz="0.0"
+        iyy="${0.0833333 * mass * (x*x + z*z)}" iyz="0.0"
+        izz="${0.0833333 * mass * (x*x + y*y)}" />
     </inertial>
   </xacro:macro>
@@ -104,6 +113,6 @@
         </geometry>
       </collision>
-      <xacro:cylinder_inertial radius="0.075" length="0.178" mass="${shoulder_mass}">
-        <origin xyz="0.0 0.0 0.0" rpy="0 0 0" />
+      <xacro:cylinder_inertial radius="0.05" length="0.124" mass="${shoulder_mass}">
+        <origin xyz="0.0 0.0 ${-0.004}" rpy="0 0 0" />
       </xacro:cylinder_inertial>
     </link>
@@ -135,6 +144,6 @@
         </geometry>
       </collision>
-      <xacro:cylinder_inertial radius="0.075" length="${-a2}" mass="${upper_arm_mass}">
-        <origin xyz="0.0 0.0 ${-a2/2.0}" rpy="0 0 0" />
+      <xacro:cylinder_inertial radius="0.05" length="0.33" mass="${upper_arm_mass}">
+        <origin xyz="0.0 0.0 ${0.33/2.0-0.048}" rpy="0 0 0" />
       </xacro:cylinder_inertial>
     </link>
@@ -166,6 +175,6 @@
         </geometry>
       </collision>
-      <xacro:cylinder_inertial radius="0.075" length="${-a3}" mass="${forearm_mass}">
-        <origin xyz="0.0 0.0 ${-a3/2.0}" rpy="0 0 0" />
+      <xacro:cylinder_inertial radius="0.04" length="0.28" mass="${forearm_mass}">
+        <origin xyz="0.0 0.0 ${0.28/2.0 - 0.037}" rpy="0 0 0" />
       </xacro:cylinder_inertial>
     </link>
@@ -197,7 +206,7 @@
         </geometry>
       </collision>
-      <xacro:cylinder_inertial radius="0.075" length="0.12" mass="${wrist_1_mass}">
+      <xacro:box_inertial x="0.0644" y="0.0796" z="0.0888" mass="${wrist_2_mass}">
         <origin xyz="0.0 ${wrist_1_length} 0.0" rpy="0 0 0" />
-      </xacro:cylinder_inertial>
+      </xacro:box_inertial>
     </link>
     <joint name="${prefix}wrist_2_joint" type="revolute">
@@ -228,7 +237,7 @@
         </geometry>
       </collision>
-      <xacro:cylinder_inertial radius="0.075" length="0.12" mass="${wrist_2_mass}">
+      <xacro:box_inertial x="0.0644" y="0.0888" z="0.0796" mass="${wrist_2_mass}">
         <origin xyz="0.0 0.0 ${wrist_2_length}" rpy="0 0 0" />
-      </xacro:cylinder_inertial>
+      </xacro:box_inertial>
     </link>
     <joint name="${prefix}wrist_3_joint" type="revolute">
