Commit message: Updated cog for ur16 how I understand the documentation
used documentation:
https://www.universal-robots.com/how-tos-and-faqs/faq/ur-faq/parameters-for-calculations-of-kinematics-and-dynamics-45257/

Note: This changes inertia for all robots as the main xacro file is changed.

File: ur_description/urdf/ur_robot.macro.xacro (robot description, xacro)
@@ -58,5 +58,5 @@
       </collision>
       <xacro:cylinder_inertial radius="${shoulder_inertia_radius}" length="${shoulder_inertia_length}" mass="${shoulder_mass}">
-        <origin xyz="0.0 0.0 0.0" rpy="0 0 0" />
+        <origin xyz="${shoulder_cog}" rpy="0 0 0" />
       </xacro:cylinder_inertial>
     </link>
@@ -88,5 +88,5 @@
       </collision>
       <xacro:cylinder_inertial radius="${upperarm_inertia_radius}" length="${upper_arm_length}" mass="${upper_arm_mass}">
-        <origin xyz="0.0 ${-upper_arm_inertia_offset} ${upper_arm_length/2.0}" rpy="0 0 0" />
+        <origin xyz="${upper_arm_cog}" rpy="0 0 0" />
       </xacro:cylinder_inertial>
     </link>
@@ -118,5 +118,5 @@
       </collision>
       <xacro:cylinder_inertial radius="${forearm_inertia_radius}" length="${forearm_length}"  mass="${forearm_mass}">
-        <origin xyz="0.0 0.0 ${forearm_length/2.0}" rpy="0 0 0" />
+        <origin xyz="${forearm_cog}" rpy="0 0 0" />
       </xacro:cylinder_inertial>
     </link>
@@ -148,5 +148,5 @@
       </collision>
       <xacro:cylinder_inertial radius="${wrist_1_inertia_radius}" length="${wrist_1_inertia_length}"  mass="${wrist_1_mass}">
-        <origin xyz="0.0 ${wrist_1_length} 0.0" rpy="0 0 0" />
+        <origin xyz="${wrist_1_cog}" rpy="0 0 0" />
       </xacro:cylinder_inertial>
     </link>
@@ -178,5 +178,5 @@
       </collision>
       <xacro:cylinder_inertial radius="${wrist_2_inertia_radius}" length="${wrist_2_inertia_length}"  mass="${wrist_2_mass}">
-        <origin xyz="0.0 0.0 ${wrist_2_length}" rpy="0 0 0" />
+        <origin xyz="${wrist_2_cog}" rpy="0 0 0" />
       </xacro:cylinder_inertial>
     </link>
@@ -208,5 +208,5 @@
       </collision>
       <xacro:cylinder_inertial radius="${wrist_3_inertia_radius}" length="${wrist_3_inertia_length}"  mass="${wrist_3_mass}">
-        <origin xyz="0.0 ${wrist_3_length - wrist_3_inertia_length/2} 0.0" rpy="${pi/2} 0 0" />
+        <origin xyz="${wrist_3_cog}" rpy="${pi/2} 0 0" />
       </xacro:cylinder_inertial>
     </link>
